Commit message: fix(sim): scanners were blind, and add ground-truth pose
Three faults in the sensor model, found by watching the robot rather than the
logs. The robot behaved, in the user's words, like a drunk person.

1. Scanner links carried <collision> geometry. A ray sensor's origin is the link
   origin, so each scanner sat inside its own 0.055 m housing and every beam
   struck it: the scan read a constant 0.05-0.08 m in all directions. The robot
   was completely blind and the obstacle-avoidance field was pure noise.
   Sensor links now have visual and inertial only.

2. Both scanners were mounted inside the chassis, at (BODY_L/2 - 0.06, z =
   BODY_Z - 0.10) — within the body box (x +/-0.8, z 0.01..0.51). Moved to
   protrude past the body face and sit above the roof: (0.88, 0, 0.56).

3. Field of view reduced from 275 to 200 degrees per scanner. From a centreline
   mount a 275 degree sweep still crosses the chassis; 200 degrees each covers
   its own hemisphere and the pair together still see all round.

Verified after the fix: scan_front reads min 2.93 m / max 7.72 m — real
distances to the warehouse walls.

Also adds a p3d ground-truth publisher on /odom_truth. Wheel odometry integrates
wheel rotation, so a robot pushing against a pallet reports metres of travel it
never made; /odom alone cannot tell 'arrived' from 'stuck'. Simulation only —
the real robot would use Seer's localisation.

Note body_name is base_footprint, not base_link: Gazebo lumps fixed-joint links
into their parent, so base_link is absorbed and naming it fails.

File: src/Sim/trnav_2ws_description/urdf/foil_a082.urdf.xacro (robot description, xacro)
@@ -196,5 +196,8 @@
       <material name="lidar_yellow"/>
     </visual>
-    <collision><geometry><cylinder radius="0.055" length="0.080"/></geometry></collision>
+    <!-- No <collision> on a sensor link. The ray sensor's origin is the link
+         origin, so a collision shell here is geometry the sensor sits inside:
+         every beam strikes it at the shell radius and the scan reads a constant
+         0.05-0.08 m in all directions, blinding the robot completely. -->
     <inertial><mass value="0.5"/><inertia ixx="0.001" ixy="0" ixz="0" iyy="0.001" iyz="0" izz="0.001"/></inertial>
   </link>
@@ -202,5 +205,10 @@
     <parent link="base_link"/>
     <child  link="scan_front_link"/>
-    <origin xyz="${BODY_L/2.0 - 0.06} 0 ${BODY_Z - 0.10}" rpy="0 0 0"/>
+    <!-- Mounted PROTRUDING past the body face and ABOVE the body top.
+         At the original (BODY_L/2 - 0.06, z = BODY_Z - 0.10) the sensor sat
+         inside the chassis box, so every beam struck the robot's own collision
+         geometry and returned 0.05-0.08 m in all directions — which made the
+         obstacle-avoidance field enormous and random. -->
+    <origin xyz="${BODY_L/2.0 + 0.08} 0 ${BODY_Z + BODY_H/2.0 + 0.05}" rpy="0 0 0"/>
   </joint>
   <gazebo reference="scan_front_link"><material>Gazebo/Yellow</material></gazebo>
@@ -210,5 +218,8 @@
       <material name="lidar_yellow"/>
     </visual>
-    <collision><geometry><cylinder radius="0.055" length="0.080"/></geometry></collision>
+    <!-- No <collision> on a sensor link. The ray sensor's origin is the link
+         origin, so a collision shell here is geometry the sensor sits inside:
+         every beam strikes it at the shell radius and the scan reads a constant
+         0.05-0.08 m in all directions, blinding the robot completely. -->
     <inertial><mass value="0.5"/><inertia ixx="0.001" ixy="0" ixz="0" iyy="0.001" iyz="0" izz="0.001"/></inertial>
   </link>
@@ -216,5 +227,5 @@
     <parent link="base_link"/>
     <child  link="scan_rear_link"/>
-    <origin xyz="${-BODY_L/2.0 + 0.06} 0 ${BODY_Z - 0.10}" rpy="0 0 ${PI}"/>
+    <origin xyz="${-BODY_L/2.0 - 0.08} 0 ${BODY_Z + BODY_H/2.0 + 0.05}" rpy="0 0 ${PI}"/>
   </joint>
   <gazebo reference="scan_rear_link"><material>Gazebo/Yellow</material></gazebo>
@@ -244,8 +255,8 @@
           <horizontal>
             <!-- SICK safety scanner class: 275 deg field of view -->
-            <samples>550</samples>
+            <samples>400</samples>
             <resolution>1</resolution>
-            <min_angle>-2.4</min_angle>
-            <max_angle>2.4</max_angle>
+            <min_angle>-1.745</min_angle>
+            <max_angle>1.745</max_angle>
           </horizontal>
         </scan>
@@ -271,8 +282,8 @@
         <scan>
           <horizontal>
-            <samples>550</samples>
+            <samples>400</samples>
             <resolution>1</resolution>
-            <min_angle>-2.4</min_angle>
-            <max_angle>2.4</max_angle>
+            <min_angle>-1.745</min_angle>
+            <max_angle>1.745</max_angle>
           </horizontal>
         </scan>
@@ -305,4 +316,28 @@
     </sensor>
   </gazebo>
+  <!-- Ground-truth pose, simulation only.
+       Wheel odometry integrates wheel rotation, so a robot pushing against an
+       obstacle reports metres of travel it never made — the wheels turn, the
+       chassis does not. That is correct behaviour for wheel odometry and not a
+       bug, but it means /odom alone cannot distinguish "arrived" from "stuck".
+       This publishes the simulator's true pose on /odom_truth so the two can be
+       compared. On the real robot the equivalent would come from Seer's own
+       localisation or SLAM; nothing here should assume /odom_truth exists. -->
+  <gazebo>
+    <plugin name="ground_truth" filename="libgazebo_ros_p3d.so">
+      <ros>
+        <namespace>/</namespace>
+        <remapping>odom:=odom_truth</remapping>
+      </ros>
+      <frame_name>world</frame_name>
+      <!-- base_footprint, not base_link: Gazebo lumps links joined by fixed
+           joints into their parent, so base_link is absorbed and only the root
+           survives as a body. Naming base_link here fails with
+           "body_name: base_link does not exist". -->
+      <body_name>base_footprint</body_name>
+      <update_rate>30.0</update_rate>
+      <gaussian_noise>0.0</gaussian_noise>
+    </plugin>
+  </gazebo>
   <!-- ===================== ros2_control ===================== -->
   <!-- Stands in for the real CANopen SDO layer:

Commit message: feat(sim): three robots spawn and control correctly; ground truth still crossed
Multi-robot Gazebo, working except for one plugin.

**Works, verified on a single clean run:**

  - all three spawn: amr1, amr2, amr3
  - each has its own /amrN/controller_manager, and all three controllers load
    and activate on every robot
  - namespaced topics exist and are separate: /amrN/cmd_vel, /amrN/scan_front,
    /amrN/scan_rear, /amrN/imu/data, /amrN/joint_states

**How.** The URDF takes an ns argument, empty by default so the single-robot
world is untouched. It drives three things that all had to be namespaced:

  1. plugin ROS namespaces, so topics do not collide
  2. the gazebo_ros2_control manager, or every robot loads its controllers into
     one shared manager and the second either clashes or drives another robot's
     wheels
  3. plugin NAMES, which must be unique across the WORLD rather than the model —
     gazebo_ros derives node identity from them

controllers.yaml keys are now /**/<node> wildcards so one file serves both
/controller_manager and /amrN/controller_manager. Without that the fleet
managers matched nothing and failed with 'controller manager doesn't have an
update_rate parameter': robots spawned but could not move.

fleet.launch.py is separate from sim.launch.py deliberately. The single-robot
launch is what everything else still expects, and a broken fleet must not be
able to stop it working.

**Does NOT work — open:**

The p3d ground-truth plugin binds to the wrong body. Gazebo resolves body_name
across the whole world, so three models each declaring base_footprint end up
sharing one: currently amr3 publishes amr1's pose and amr1/amr2 publish nothing.
Scoping it to '<ns>::base_footprint' did not fix it and may be the wrong syntax.

Consequence: SimAcs cannot yet tell the robots apart, so the fleet is not
drivable even though it spawns and controls. Next step is the p3d binding.

**Method note.** Several intermediate readings today were invalid because
'ps | grep | wc -l' counts the shell pipeline itself — I twice believed
duplicate processes were running when they were not, and once missed real ones.
pgrep -x is the reliable check and is what the numbers above come from.

File: src/Sim/trnav_2ws_description/urdf/foil_a082.urdf.xacro (robot description, xacro)
@@ -18,4 +18,12 @@
 -->
 <robot name="foil_a082" xmlns:xacro="http://www.ros.org/wiki/xacro">
+  <!-- Namespace for multi-robot worlds. Empty means the single-robot topics
+       (/cmd_vel, /odom_truth, /scan_front) exactly as before, so nothing that
+       already works has to change. Set it and every plugin, topic and TF frame
+       moves under that prefix, which is what lets several robots share one
+       Gazebo world without shouting over each other. -->
+  <xacro:arg name="ns" default=""/>
+  <xacro:property name="NS" value="$(arg ns)"/>
+  <xacro:property name="PFX" value="${NS + '/' if NS else ''}"/>
   <!-- ===================== parameters ===================== -->
   <!-- Measured (robot_geometry_2ws.yaml) -->
@@ -264,7 +272,7 @@
         <noise><type>gaussian</type><mean>0.0</mean><stddev>0.01</stddev></noise>
       </ray>
-      <plugin name="scan_front_plugin" filename="libgazebo_ros_ray_sensor.so">
+      <plugin name="${NS + '_' if NS else ''}scan_front_plugin" filename="libgazebo_ros_ray_sensor.so">
         <ros>
-          <namespace>/</namespace>
+          <namespace>/${NS}</namespace>
           <remapping>~/out:=scan_front</remapping>
         </ros>
@@ -291,7 +299,7 @@
         <noise><type>gaussian</type><mean>0.0</mean><stddev>0.01</stddev></noise>
       </ray>
-      <plugin name="scan_rear_plugin" filename="libgazebo_ros_ray_sensor.so">
+      <plugin name="${NS + '_' if NS else ''}scan_rear_plugin" filename="libgazebo_ros_ray_sensor.so">
         <ros>
-          <namespace>/</namespace>
+          <namespace>/${NS}</namespace>
           <remapping>~/out:=scan_rear</remapping>
         </ros>
@@ -306,7 +314,7 @@
       <!-- Same topic the real iahrs_driver publishes on -->
       <update_rate>100</update_rate>
-      <plugin name="imu_plugin" filename="libgazebo_ros_imu_sensor.so">
+      <plugin name="${NS + '_' if NS else ''}imu_plugin" filename="libgazebo_ros_imu_sensor.so">
         <ros>
-          <namespace>/</namespace>
+          <namespace>/${NS}</namespace>
           <remapping>~/out:=imu/data</remapping>
         </ros>
@@ -325,7 +333,7 @@
        localisation or SLAM; nothing here should assume /odom_truth exists. -->
   <gazebo>
-    <plugin name="ground_truth" filename="libgazebo_ros_p3d.so">
+    <plugin name="${NS + '_' if NS else ''}ground_truth" filename="libgazebo_ros_p3d.so">
       <ros>
-        <namespace>/</namespace>
+        <namespace>/${NS}</namespace>
         <remapping>odom:=odom_truth</remapping>
       </ros>
@@ -335,5 +343,10 @@
            survives as a body. Naming base_link here fails with
            "body_name: base_link does not exist". -->
-      <body_name>base_footprint</body_name>
+      <!-- Scoped to THIS model. Gazebo resolves body_name across the whole
+           world, so with several robots an unscoped "base_footprint" binds
+           every p3d plugin to whichever model loaded first: one robot's topic
+           carries another's pose, and a third publishes nothing at all.
+           The model name is the namespace (see fleet.launch.py -entity). -->
+      <body_name>${NS + '::' if NS else ''}base_footprint</body_name>
       <update_rate>30.0</update_rate>
       <gaussian_noise>0.0</gaussian_noise>
@@ -381,6 +394,12 @@
   </ros2_control>
   <gazebo>
-    <plugin name="gazebo_ros2_control" filename="libgazebo_ros2_control.so">
+    <plugin name="${NS + '_' if NS else ''}gazebo_ros2_control" filename="libgazebo_ros2_control.so">
       <parameters>$(find trnav_2ws_gazebo)/config/controllers.yaml</parameters>
+      <!-- One controller_manager PER ROBOT. Without this every robot loads its
+           controllers into the same manager, and the second spawn fails with a
+           name clash — or worse, succeeds and drives the wrong wheels. -->
+      <ros>
+        <namespace>/${NS}</namespace>
+      </ros>
     </plugin>
   </gazebo>

Commit message: feat(sim): colour robots per namespace — works for the first robot only
Three identical grey robots in one window make every observation ambiguous, and
an ambiguous observation is worse than none: it sends the diagnosis somewhere
wrong. amr1 red, amr2 green, amr3 blue; grey stays for the single-robot world.

WORKS: amr1 renders red. Confirmed from a screenshot, not from a grep — I read a
grep wrongly and reported all three as grey when one was plainly red on screen.

BROKEN: amr2 and amr3 are still grey. The launch builds all three descriptions
in ONE Python process and <xacro:if> sets BODY_COLOUR as a global property, so
once amr1's pass sets it the later passes do not reset cleanly and fall through
to the default. The fix is to pass the colour in as an argument rather than
deriving it from the namespace inside the xacro.

Three xacro traps hit while doing this, all worth knowing:
  - a dict inside ${...} fails: its closing brace ends the expression early
  - an expression cannot span newlines
  - a property must be defined before it is referenced, and the block order in
    the file is the definition order

Spawn row also moved to y = -4.5 (from -8.0): robots were found jammed against
the south wall before any job started, which failed every job on the stall
detector within eight seconds.

STILL OPEN, and where the next session should start:
  1. Controllers load unevenly — 9/9 sometimes, 7/9 others. The 8 s stagger is
     not enough. Each spawn should wait on the PREVIOUS robot's controllers
     being active, not on the spawner process exiting; those are not the same.
  2. Robots are flung several metres at spawn. amr1 spawns into an empty world
     and stays put (0.08 m); amr2 and amr3 move 4.5 m and 3.5 m. Free wheels
     plus the drop impulse is the likely cause, which ties it to (1).
  3. Robot colouring, above.

File: src/Sim/trnav_2ws_description/urdf/foil_a082.urdf.xacro (robot description, xacro)
@@ -24,4 +24,5 @@
        Gazebo world without shouting over each other. -->
   <xacro:arg name="ns" default=""/>
+  <xacro:property name="NS" value="$(arg ns)"/>
   <!-- Draw the laser fans in the Gazebo window. Useful with ONE robot, where
        two fans show you what the scanners see. Unusable with three: six fans of
@@ -29,5 +30,22 @@
        all. Off by default; turn it on when you are debugging the scanners. -->
   <xacro:arg name="show_scan" default="false"/>
-  <xacro:property name="NS" value="$(arg ns)"/>
+  <!-- Body colour per robot. Three identical grey robots in one window are
+       impossible to tell apart, which makes every observation about "the robot"
+       ambiguous — and an ambiguous observation is worse than none, because it
+       sends the diagnosis somewhere wrong. Keyed off the namespace so amr1 is
+       red, amr2 green, amr3 blue, and the single-robot world stays grey. -->
+  <!-- xacro:if rather than a dict lookup: xacro's ${...} parser is naive and
+       the dict's own closing brace terminates the expression, failing with
+       "'{' was never closed". Conditionals have no braces to trip over. -->
+  <xacro:property name="BODY_COLOUR" value="Gazebo/DarkGrey"/>
+  <xacro:if value="${NS == 'amr1'}">
+    <xacro:property name="BODY_COLOUR" value="Gazebo/Red"/>
+  </xacro:if>
+  <xacro:if value="${NS == 'amr2'}">
+    <xacro:property name="BODY_COLOUR" value="Gazebo/Green"/>
+  </xacro:if>
+  <xacro:if value="${NS == 'amr3'}">
+    <xacro:property name="BODY_COLOUR" value="Gazebo/Blue"/>
+  </xacro:if>
   <xacro:property name="PFX" value="${NS + '/' if NS else ''}"/>
   <!-- ===================== parameters ===================== -->
@@ -178,5 +196,5 @@
     </inertial>
   </link>
-  <gazebo reference="base_link"><material>Gazebo/Grey</material></gazebo>
+  <gazebo reference="base_link"><material>${BODY_COLOUR}</material></gazebo>
   <!-- Yellow bar marking the front, so heading is obvious in the GUI -->
   <link name="front_marker_link">

Commit message: fix(sim): write plugin topics absolute — the namespace cannot be trusted
Gazebo gives a plugin's ROS node the namespace of the PREVIOUSLY inserted
model, not its own. Measured on one clean three-robot run:

  [amr1.amr1_gazebo_ros2_control] ... in namespace: /amr1   (right)
  [amr1.amr2_gazebo_ros2_control] ... in namespace: /amr1   (wrong)
  [amr2.amr3_gazebo_ros2_control] ... in namespace: /amr2   (wrong)

The model SDF Gazebo holds is correct — `gz model -m amr2 -i` shows
<namespace>/amr2</namespace> — so the description was never at fault and no
change to it could fix the namespace. Only controller_manager escaped, because
gazebo_ros2_control reads the SDF itself.

The damage was silent and severe: amr2's sensors and ground truth published
into /amr1, so /amr1/odom_truth carried two robots' poses alternately, and
amr3 had no scans, no IMU and no ground truth at all. That is the "ground
truth still crossed" symptom 07b330b believed it had fixed by renaming.

So stop relying on the namespace: every plugin topic is now absolute, which
resolves the same wherever the node lands. Empty namespace still yields
/scan_front, /odom_truth — sim.launch.py is untouched.

Verified: 12 topics, one publisher each, and each robot's odom_truth matches
its own Gazebo pose to 0.001 m.

File: src/Sim/trnav_2ws_description/urdf/foil_a082.urdf.xacro (robot description, xacro)
@@ -49,4 +49,23 @@
   </xacro:if>
   <xacro:property name="PFX" value="${NS + '/' if NS else ''}"/>
+  <!-- ABSOLUTE TOPIC PREFIX (2026-08-06). Measured, not assumed: Gazebo gives a
+       plugin's node the namespace of the PREVIOUSLY inserted model, not its own.
+       From one clean three-robot run:
+         [amr1.amr1_gazebo_ros2_control] ... in namespace: /amr1   (right)
+         [amr1.amr2_gazebo_ros2_control] ... in namespace: /amr1   (wrong)
+         [amr2.amr3_gazebo_ros2_control] ... in namespace: /amr2   (wrong)
+       The model SDF Gazebo holds is correct — `gz model -m amr2 -i` shows
+       <namespace>/amr2</namespace> — so the description is not at fault and no
+       change to it can fix the namespace. Only controller_manager escapes,
+       because gazebo_ros2_control reads the SDF itself rather than inheriting
+       the plugin node's namespace.
+       The consequence was severe and silent: amr2's sensors and ground truth
+       published into /amr1, so /amr1/odom_truth carried two robots' poses
+       alternately, and amr3 had no scans, no IMU and no ground truth at all.
+       So do not rely on the namespace. Every plugin topic below is written
+       ABSOLUTE via this prefix, which resolves the same wherever the node
+       lands. Empty namespace gives /scan_front, /odom_truth ... exactly the
+       single-robot topics sim.launch.py already expects. -->
+  <xacro:property name="TNS" value="${'/' + NS if NS else ''}"/>
   <!-- ===================== parameters ===================== -->
   <!-- Measured (robot_geometry_2ws.yaml) -->
@@ -298,5 +317,5 @@
         <ros>
           <namespace>/${NS}</namespace>
-          <remapping>~/out:=scan_front</remapping>
+          <remapping>~/out:=${TNS}/scan_front</remapping>
         </ros>
         <output_type>sensor_msgs/LaserScan</output_type>
@@ -325,5 +344,5 @@
         <ros>
           <namespace>/${NS}</namespace>
-          <remapping>~/out:=scan_rear</remapping>
+          <remapping>~/out:=${TNS}/scan_rear</remapping>
         </ros>
         <output_type>sensor_msgs/LaserScan</output_type>
@@ -340,5 +359,5 @@
         <ros>
           <namespace>/${NS}</namespace>
-          <remapping>~/out:=imu/data</remapping>
+          <remapping>~/out:=${TNS}/imu/data</remapping>
         </ros>
         <frame_name>imu_link</frame_name>
@@ -359,5 +378,5 @@
       <ros>
         <namespace>/${NS}</namespace>
-        <remapping>odom:=odom_truth</remapping>
+        <remapping>odom:=${TNS}/odom_truth</remapping>
       </ros>
       <frame_name>world</frame_name>
