Commit message: feat(sim): give the robot its two docking cameras
Mirrors the docking project, which carries a RealSense on each side. They face
SIDEWAYS because the robot crabs into a dock: the machine is beside it, never
ahead. That is also why the drive controller holds its aisle heading on a spur.

Two details that each cost a restart to find:

  The remapping source is the CAMERA NAME, not ~. gazebo_ros_camera publishes
  on "<camera_name>/image_raw" relative to its node, so a "~/image_raw" rule
  never matches and the absolute target is silently not applied. Gazebo's
  namespace shift then put amr2's cameras onto /amr1 and lost amr3's entirely:
  /amr1/dock_camera_left/image_raw had 2 publishers and /amr3 had none.

  Mounted flush with the body edge. Moving them inboard looks like it buys
  working distance and instead puts the robot's own chassis in the bottom third
  of the frame — the body half-width is 0.45 and its top only 0.04 m below the
  lens, so the camera stares across its own roof and the marker is clipped from
  below.

Verified: six topics, one publisher each, and the marker fully in frame from
the approach point all the way to the docked standoff.

File: src/Sim/trnav_2ws_description/urdf/foil_a082.urdf.xacro (robot description, xacro)
@@ -396,4 +396,68 @@
     </plugin>
   </gazebo>
+  <!-- ===================== docking cameras ===================== -->
+  <!-- TWO cameras, one per side, optical axis along body +/-y.
+       Mounting mirrors the docking project (docking_gui_dist), which carries a
+       RealSense on each side: left_link (0, +0.34, 0.16) yaw +pi/2, right_link
+       the mirror of it. Scaled to this chassis, which is 0.9 m wide.
+       They face SIDEWAYS because the robot crabs into a dock: the machine is
+       beside it, never ahead. That is also why the drive controller holds its
+       aisle heading on a docking spur — turning to face the machine would swing
+       the marker out of both cameras' view. -->
+  <!-- AT THE BODY EDGE, flush. Moving these inboard looked like it would buy
+       working distance for the lens, and instead put the robot's own chassis in
+       the bottom third of the frame: the body half-width is 0.45 and its top is
+       only 0.04 m below the lens, so from 0.20 m the camera stares across its
+       own roof and the marker is clipped from below. Flush with the edge, the
+       body is behind the lens and cannot occlude anything.
+       The cost is that at the docked standoff the lens is only 0.16 m from the
+       marker and sees 0.22 m of width — which is what sets the marker size. -->
+  <xacro:property name="CAM_Y" value="0.46"/>
+  <xacro:property name="CAM_Z" value="0.55"/>
+  <xacro:macro name="dock_camera" params="side y yaw">
+    <link name="cam_${side}_link">
+      <visual>
+        <geometry><box size="0.03 0.10 0.03"/></geometry>
+        <material name="imu_green"/>
+      </visual>
+      <inertial><mass value="0.1"/><inertia ixx="1e-4" ixy="0" ixz="0" iyy="1e-4" iyz="0" izz="1e-4"/></inertial>
+    </link>
+    <joint name="cam_${side}_joint" type="fixed">
+      <parent link="base_link"/>
+      <child  link="cam_${side}_link"/>
+      <origin xyz="0 ${y} ${CAM_Z}" rpy="0 0 ${yaw}"/>
+    </joint>
+    <gazebo reference="cam_${side}_link">
+      <sensor type="camera" name="dock_cam_${side}">
+        <update_rate>15.0</update_rate>
+        <visualize>false</visualize>
+        <camera>
+          <!-- ~69 deg horizontal, the D435 colour stream. The docking
+               observation model assumes a 55 deg half-angle; this is wider,
+               so what the controller is told it can see, it really can. -->
+          <horizontal_fov>1.204</horizontal_fov>
+          <image><width>640</width><height>480</height><format>R8G8B8</format></image>
+          <clip><near>0.05</near><far>30.0</far></clip>
+        </camera>
+        <plugin name="${NS + '_' if NS else ''}dock_cam_${side}" filename="libgazebo_ros_camera.so">
+          <ros>
+            <namespace>/${NS}</namespace>
+            <!-- Source name is the CAMERA NAME, not ~. gazebo_ros_camera
+                 publishes on "<camera_name>/image_raw" relative to its node,
+                 so a "~/image_raw" rule never matches and the absolute target
+                 is silently not applied — which let Gazebo's namespace shift
+                 put amr2's cameras onto /amr1 and lose amr3's entirely.
+                 Measured: /amr1/dock_camera_left/image_raw had 2 publishers. -->
+            <remapping>dock_camera_${side}/image_raw:=${TNS}/dock_camera_${side}/image_raw</remapping>
+            <remapping>dock_camera_${side}/camera_info:=${TNS}/dock_camera_${side}/camera_info</remapping>
+          </ros>
+          <camera_name>dock_camera_${side}</camera_name>
+          <frame_name>${NS + '_' if NS else ''}cam_${side}_link</frame_name>
+        </plugin>
+      </sensor>
+    </gazebo>
+  </xacro:macro>
+  <xacro:dock_camera side="left"  y="${CAM_Y}"  yaw="${PI2}"/>
+  <xacro:dock_camera side="right" y="${-CAM_Y}" yaw="${-PI2}"/>
   <!-- ===================== ros2_control ===================== -->
   <!-- Stands in for the real CANopen SDO layer:

Commit message: test(sim/description): 조향 한계 90°→115° (크랩 시 하드스톱 회피)
Both drive wheels are on the centreline, so a pure sideways crab — exactly what
docking does — demands both wheels at +/-90 deg. At a 90 deg limit that IS the
hard stop, and docking froze there: two robots reached 0.45 m range against a
0.65 m target, sat still for 90 s and timed out. The docks that succeeded were
the ones a few degrees OFF parallel, where the demand stayed inside travel.

115 deg leaves 25 deg of margin at the crab. NOTE this diverges from every
steer_limit_deg in the repo (all 90.0) including spin_params.yaml, which this
model's header cites as its source — deliberately, pending confirmation.

File: src/Sim/trnav_2ws_description/urdf/foil_a082.urdf.xacro (robot description, xacro)
@@ -76,5 +76,15 @@
   <xacro:property name="WHEEL_R" value="0.125"/>
   <xacro:property name="WHEEL_W" value="0.080"/>
-  <xacro:property name="STEER_LIMIT" value="1.5707963267948966"/>  <!-- +/-90 deg -->
+  <!-- TEST 2026-08-07: +/-115 deg, not 90.
+       Both drive wheels are on the centreline, so a pure sideways crab — which
+       is exactly what docking does — needs both wheels at +/-90 deg. At a 90 deg
+       limit that is the HARD STOP, and docking froze there: two robots reached
+       range 0.45 m against a 0.65 m target, sat perfectly still for 90 s and
+       timed out. The docks that succeeded were the ones a few degrees OFF
+       parallel, where the demand stays inside travel.
+       115 deg leaves 25 deg of margin at the crab. Session memory records the
+       real limit being changed from 90 to 115; if this run docks cleanly that
+       is confirmed, and if not the limit was never the problem. -->
+  <xacro:property name="STEER_LIMIT" value="2.0071286397934789"/>  <!-- +/-115 deg -->
   <!-- PLACEHOLDER - change here and the whole model follows -->
   <xacro:property name="BODY_L" value="1.600"/>

Commit message: fix(csm): give-way that actually gives way, and an instrument that can see contact
Four defects in the give-way handshake, each found in Gazebo and each measured
before and after. Unit tests did not catch any of them and passed throughout.

1. A yielder aimed its lay-by by heading alone. A robot standing ON an aisle
   but turned toward its station read as travelling north-south, so its
   candidates became x-offsets from the far cross aisle — 14.4 m away, on the
   far side of the robot it was yielding to. `_sidestep_target` now offers both
   axes with the heading only ORDERING them, and rejects any candidate the
   partner blocks. Cost of the bug: amr1 and amr2 deadlocked 2.25 m apart,
   two jobs failed at YIELD_LIMIT.

2. "Both candidates fouled" returned a fouled one anyway, on the reasoning that
   moving away beats driving at it. Where the partner is between us and that
   whole side — the only case that reaches there — the furthest candidate is the
   one deepest THROUGH it. It now reports None, and `SimAcs.cannot_yield` hands
   the duty to the robot that does have room. One hand-over per encounter.

3. `_off_the_road` asked what KIND of place the robot was in, not whether its
   body was clear of the lane. `_in_a_bay` is any marker within 3.0 m, and a bay
   circle on the south row reaches 1.0 m from the south aisle — so a robot could
   answer "already clear — you may pass" without moving and still be in the way.
   It now measures distance to each through lane against what the robot needs
   from that lane AT ITS CURRENT HEADING: a 1.6 x 0.9 m body reaches 0.45 m
   across a lane when parallel and 0.80 m when square on. Cost of the bug:
   amr3/amr4 contact at 0.00 m, and later 0.16 m with a flat rule.

4. The branch above then did `return False`, which hands the tick back to the
   work path — so the yielder resumed driving to its own goal the moment it
   declared itself clear. Safe while the test meant "parked in a bay"; a
   bouncing robot once the test depended on live pose. Measured: amr2 announced
   "already clear" 29 times in 10.7 minutes and no stand-aside ever completed,
   while amr1 held at v=0.00 as the passer. A give-way is a promise to stay put;
   it now stops and holds.

Also: a lay-by is unreachable whoever is standing in it, not only the partner —
and the robot most likely to be in it is the one QUEUEING for that encounter,
since `_yielder_ahead` holds it back and where it holds is often the lay-by.

Tools/contact_meter/ measures body separation from OUTSIDE this code. Contact
writes no log line, which is how a run with a collision in it was reported as
clean. It imports nothing from csm and computes oriented-rectangle separation
itself, because on 2026-08-10 a meter built on the traffic layer's own capsule
model reported "no contact" through an overlap.

Fleet colour is now keyed off the leg (plant.ROBOT_SEGMENT) rather than three
hardcoded robot names, so segment A is red, B green, C blue at any fleet size.
At robots:=5 amr4 and amr5 were falling through to the single-robot grey.

4-robot Gazebo, 26.4 min, against the pre-change baseline over 61.5 min:
    deliveries/min      1.0 -> 1.3
    give-ways completed 54% -> 79%
    yield timeouts        2 -> 0
    contacts              1 -> 0

KNOWN NOT FIXED, all reproduced and diagnosed, none of them regressions:
  - a yielder that reports itself already clear never sets `_yield_since`, so
    YIELD_LIMIT cannot fire and the hold is unbounded
  - slitter dock pitch is 2.00 m where every other port pair in the plant uses
    2.40 m; 2.02 m is the minimum for a robot to turn beside a parked one, so
    adjacent slitter docks cannot both be used
  - `plant.segment_for_job` ignores each segment's `buffer` list, so every
    divert-to-rack job is rejected and retried at 2/s
  - the dispatcher grants one permit at a time to the oldest job, so an
    unservable job starves work for an idle robot on another leg
  - one encounter per robot (this commit) removes the three-way cycle but
    leaves a refused robot with no recourse; at robots:=5 it produced 22
    no-op deadlock-breaker calls

File: src/Sim/trnav_2ws_description/urdf/foil_a082.urdf.xacro (robot description, xacro)
@@ -30,20 +30,35 @@
        all. Off by default; turn it on when you are debugging the scanners. -->
   <xacro:arg name="show_scan" default="false"/>
-  <!-- Body colour per robot. Three identical grey robots in one window are
-       impossible to tell apart, which makes every observation about "the robot"
-       ambiguous — and an ambiguous observation is worse than none, because it
-       sends the diagnosis somewhere wrong. Keyed off the namespace so amr1 is
-       red, amr2 green, amr3 blue, and the single-robot world stays grey. -->
+  <!-- Body colour per LEG, not per robot. Identical grey robots in one window
+       are impossible to tell apart, which makes every observation about "the
+       robot" ambiguous — and an ambiguous observation is worse than none,
+       because it sends the diagnosis somewhere wrong. What you need to read off
+       the window is which leg of the material flow a robot is serving, so that
+       is what the colour carries: A red, B green, C blue. Robots on the same
+       leg are the same colour on purpose — they are interchangeable, and the
+       CSM treats them that way. The single-robot world passes no segment and
+       stays grey.
+       KEYED OFF THE SEGMENT, NOT THE NAME. It used to be three xacro:if cases
+       on the namespace — amr1 red, amr2 green, amr3 blue — and every robot
+       past the third fell through to the default. At robots:=5 that put amr4
+       and amr5 on segment C in DarkGrey, the same grey the single-robot world
+       uses, so the window showed four colours for three legs. This is the same
+       failure fleet.launch.py records against its own hand-written fleet tuple:
+       a list written out by hand caps the fleet at the length of the list. The
+       leg map lives in csm/plant.py ROBOT_SEGMENT and the launch passes it in,
+       so this stays right at the deck's full ten. -->
   <!-- xacro:if rather than a dict lookup: xacro's ${...} parser is naive and
        the dict's own closing brace terminates the expression, failing with
        "'{' was never closed". Conditionals have no braces to trip over. -->
+  <xacro:arg name="segment" default=""/>
+  <xacro:property name="SEGMENT" value="$(arg segment)"/>
   <xacro:property name="BODY_COLOUR" value="Gazebo/DarkGrey"/>
-  <xacro:if value="${NS == 'amr1'}">
+  <xacro:if value="${SEGMENT == 'A'}">
     <xacro:property name="BODY_COLOUR" value="Gazebo/Red"/>
   </xacro:if>
-  <xacro:if value="${NS == 'amr2'}">
+  <xacro:if value="${SEGMENT == 'B'}">
     <xacro:property name="BODY_COLOUR" value="Gazebo/Green"/>
   </xacro:if>
-  <xacro:if value="${NS == 'amr3'}">
+  <xacro:if value="${SEGMENT == 'C'}">
     <xacro:property name="BODY_COLOUR" value="Gazebo/Blue"/>
   </xacro:if>
